Commit message: HW1: modified to correct meshes

File: armando_description/urdf/arm.urdf (robot description, URDF)
Before this commit: robot arm, 17 links, 16 joints
Links:
- link crawer_left: geometry collision box size=0.063 0.031 0.041; visual mesh filename=package://armando_description/meshes/the_crawer.stl scale=0.001 0.001 0.001
- link crawer_right: geometry collision box size=0.063 0.031 0.041; visual mesh filename=package://armando_description/meshes/the_crawer.stl scale=0.001 0.001 0.001
